File: KiCad Project/NavigationSystem.kicad_pcb (KiCad board)
At the start: 4 copper layers, 125.8 x 96.7 mm, 92 parts, among them J1 Screw_Terminal_01x02, J10 Conn_01x03, J11 Conn_01x03, J15 Conn_01x04, J16 Conn_01x03, J17 Conn_01x03, J18 Conn_01x03, J2 SWD, J3 Conn_01x04, J4 5-1814832-1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

Commit message: power modules updated
reverse polarity protection
Parts:
- added D10: GREEN, LED_SMD:LED_0603_1608Metric, F.Cu at (127.4, 65.2)
- added D11: ZMMxx, Diode_SMD:D_MiniMELF, F.Cu at (126.2, 62.7)
- added D6: BLUE, LED_SMD:LED_0603_1608Metric, F.Cu at (90.5, 64.0)
- added D7: RED, LED_SMD:LED_0603_1608Metric, F.Cu at (127.4, 67.4)
- added D8: RED, LED_SMD:LED_0603_1608Metric, F.Cu at (74.2, 77.1)
- added R20: 100r, Resistor_SMD:R_0603_1608Metric, F.Cu at (130.6, 62.8)
- added R21: 1k5, Resistor_SMD:R_0603_1608Metric, F.Cu at (130.7, 67.4)
- added R22: 1k5, Resistor_SMD:R_0603_1608Metric, F.Cu at (130.6, 65.2)
- added R23: 1k5, Resistor_SMD:R_0603_1608Metric, F.Cu at (93.9, 64.0)
- added R24: 1k5, Resistor_SMD:R_0603_1608Metric, F.Cu at (76.2, 77.1)
- C1, C26, C32, C33, C34: footprint Capacitor_SMD:C_1206_3216Metric -> Capacitor_SMD:C_0603_1608Metric
- C17, C18: footprint Capacitor_SMD:C_0603_1608Metric -> Capacitor_SMD:C_0402_1005Metric
- D1, D9: footprint Diode_SMD:D_SOD-123 -> Diode_SMD:D_0603_1608Metric
- F1: footprint Fuse:Fuse_1206_3216Metric -> Fuse:Fuse_0603_1608Metric
- R12, R13: footprint Resistor_SMD:R_0603_1608Metric -> Resistor_SMD:R_0402_1005Metric
- moved R16 6.22 mm to (103.5, 74.5)
- moved C3 6.15 mm to (68.5, 79.2), turned to 270 degrees
- moved R12 5.04 mm to (46.0, 101.4), turned to 0 degrees
- moved C33 3.73 mm to (103.5, 72.4)
- moved C2 3.32 mm to (71.2, 79.2), turned to 270 degrees
- moved D2 2.98 mm to (73.9, 65.9), turned to 90 degrees
- moved C1 2.47 mm to (80.7, 68.3)
- moved C26 2.17 mm to (90.5, 66.1)
- moved R17 2.08 mm to (97.9, 78.4)
- moved C32 1.81 mm to (97.9, 66.1)
- moved C18 1.41 mm to (46.1, 103.6)
- moved C20 1.32 mm to (28.0, 101.4)
- moved C17 1.13 mm to (46.1, 102.4)
- moved C34 1.10 mm to (92.0, 76.7)
- moved D9 0.87 mm to (97.9, 76.8)
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Connections:
- net VS_1 renamed Net-(2920L700SLPR1-Pad1)
- Q2 pad 1: GND -> Net-(D11-Pad2)
Routing:
- net GND: track 155.9 -> 127.3 mm, vias 62 -> 60
- net VS: track 18.0 -> 39.1 mm
- net Net-(2920L700SLPR1-Pad1): track 7.58 -> 17.6 mm
- net Net-(D11-Pad2): track 0.00 -> 6.86 mm
- net +3V3: track 79.8 -> 85.9 mm, vias 31 -> 28
- net Net-(C33-Pad1): track 15.5 -> 11.2 mm
- net Regulated12V: track 128.6 -> 131.8 mm
- net BUCK_SW: track 9.65 -> 12.8 mm
- net GPS_NRST_NAVC: track 5.80 -> 3.09 mm
- net Net-(D8-Pad1): track 0.00 -> 2.03 mm
- net Net-(D6-Pad1): track 0.00 -> 1.80 mm
- net Net-(D7-Pad1): track 0.00 -> 1.66 mm
- net Net-(D10-Pad1): track 0.00 -> 1.59 mm
- net Net-(D1-Pad1): track 4.80 -> 6.26 mm
- net BUCK_IN: track 8.78 -> 10.2 mm
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Other:
- board text added: "IMU"
- board text removed: "FXOS8700CQ"
